File: hardware/robot-carrier/_restore_backup_2026-08-17T17-35-53-814/robot-carrier.kicad_sch (KiCad schematic)
At the start: 36 parts, among them J1 6S BATTERY INPUT, J10 M1 JGA25-2430-CE, J100 PROTECTED 6S BATTERY, J101 EXTERNAL BUCK 5V OUTPUT, J11 M2 JGA25-2430-CE, J12 M3 JGA25-2430-CE, J13 M4 JGA25-2430-CE, J2 BUCK INPUT 24V, J20 SERVO 1, J21 SERVO 2, J22 SERVO 3, J23 SERVO 4, J3 BUCK OUTPUT 5V, J30 IMU I2C, J40 GA25 L298N LOGIC, J41 GA25 L298N POWER

Commit message: updated to none cropper pour
Parts:
- C1: value HRK 2200uF 63V CD288 -> 470uF 63V; footprint Capacitor_THT:CP_Radial_D18.0mm_P7.50mm -> Capacitor_THT:CP_Radial_D10.0mm_P5.00mm; LCSC C2960335 -> C51953331
- J1, J2, J3: LCSC C8404 -> C500021
- J40: LCSC C52016391 -> (none)
- R1, R10, R11, R12, R2, R3, R4, R7, R8, R9: LCSC C17414 -> C17902
Changed lines of the file:
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@@
 			)
 		)
-		(property "LCSC" "C8404"
+		(property "LCSC" "C500021"
 			(at 76.2 25.4 0)
 				(effects
@@
 			)
 		)
-			(property "Value" "HRK 2200uF 63V CD288"
+		(property "Value" "470uF 63V"
 			(at 137.16 29.21 0)
 				(effects
@@
 			)
 		)
-			(property "Footprint" "Capacitor_THT:CP_Radial_D18.0mm_P7.50mm"
+		(property "Footprint" "Capacitor_THT:CP_Radial_D10.0mm_P5.00mm"
 			(at 137.16 25.4 0)
 				(effects
@@
 			)
 		)
-			(property "Description" "HRK 2200uF 63V CD288, D18xL32mm"
+		(property "Description" "470uF 63V"
 			(at 137.16 25.4 0)
 				(effects
@@
 			)
 		)
-			(property "LCSC" "C2960335"
+		(property "LCSC" "C51953331"
 			(at 137.16 25.4 0)
 				(effects
@@
 			)
 		)
-		(property "LCSC" "C8404"
+		(property "LCSC" "C500021"
 			(at 45.72 44.45 0)
 				(effects
@@
 			)
 		)
-		(property "LCSC" "C8404"
+		(property "LCSC" "C500021"
 			(at 137.16 44.45 0)
 				(effects
@@
 			)
 		)
-		(property "LCSC" "C52016391"
-			(at 100.33 180.34 0)
-			(effects
-				(font
-					(size 1.27 1.27)
-				)
-				(hide yes)
-			)
-		)
 		(pin "1")
 		(pin "2")
@@
 			)
 		)
-		(property "LCSC" "C17414"
+		(property "LCSC" "C17902"
 			(at 299.72 30.48 0)
 				(effects
@@
 			)
 		)
-		(property "LCSC" "C17414"
+		(property "LCSC" "C17902"
 			(at 299.72 41.91 0)
 				(effects
@@
 			)
 		)
-		(property "LCSC" "C17414"
+		(property "LCSC" "C17902"
 			(at 299.72 54.61 0)
 				(effects
@@
 			)
 		)
-		(property "LCSC" "C17414"
+		(property "LCSC" "C17902"
 			(at 299.72 66.04 0)
 				(effects
@@
 			)
 		)
-		(property "LCSC" "C17414"
+		(property "LCSC" "C17902"
 			(at 299.72 101.6 0)
 				(effects
@@
 			)
 		)
-		(property "LCSC" "C17414"
+		(property "LCSC" "C17902"
 			(at 299.72 114.3 0)
 				(effects
@@
 			)
 		)
-		(property "LCSC" "C17414"
+		(property "LCSC" "C17902"
 			(at 299.72 125.73 0)
 				(effects
@@
 			)
 		)
-		(property "LCSC" "C17414"
+		(property "LCSC" "C17902"
 			(at 299.72 138.43 0)
 				(effects
@@
 			)
 		)
-		(property "LCSC" "C17414"
+		(property "LCSC" "C17902"
 			(at 299.72 149.86 0)
 				(effects
@@
 			)
 		)
-		(property "LCSC" "C17414"
+		(property "LCSC" "C17902"
 			(at 299.72 162.56 0)
 				(effects
