File: hardware/robot-carrier/robot-carrier.kicad_sch (KiCad schematic)
At the start: 36 parts, among them J1 6S BATTERY INPUT, J10 M1 JGA25-2430-CE, J100 PROTECTED 6S BATTERY, J101 EXTERNAL BUCK 5V OUTPUT, J11 M2 JGA25-2430-CE, J12 M3 JGA25-2430-CE, J13 M4 JGA25-2430-CE, J2 BUCK INPUT 24V, J20 SERVO 1, J21 SERVO 2, J22 SERVO 3, J23 SERVO 4, J3 BUCK OUTPUT 5V, J30 IMU I2C, J40 GA25 L298N LOGIC, J41 GA25 L298N POWER

Commit message: Reroute carrier board
Parts:
- added D2: SMAJ5.0A, Diode_SMD:D_SMA, symbol RobotCarrier:D_TVS
- added F102: PPTC 0.75A 6V, Fuse:Fuse_1812_4532Metric, symbol RobotCarrier:Fuse
- added R13, R14: 470R, Custom:R_1206_HAND, symbol RobotCarrier:R
- JPI1: value RPI4B POWER UART -> RPI4B UART (GND / TX / RX); footprint Custom:PI_REMOTE_1X06_MALE -> Custom:DUPONT_MALE_1X03; symbol RobotCarrier:Conn_01x06 -> RobotCarrier:Conn_01x03
Connections:
- net +5V: now also F102.1 (Pin_1); no longer JESP1.15 (Pin_15), JPI1.1 (Pin_1), JPI1.2 (Pin_2)
- net GND: now also JPI1.1 (Pin_1), D2.2 (Pin_2); no longer JPI1.3 (Pin_3), JPI1.4 (Pin_4)
- net PI_UART_RX_3V3: now also JPI1.3 (Pin_3), R14.2 (Pin_2); no longer JESP1.19 (Pin_19), JPI1.6 (Pin_6)
- net PI_UART_TX_3V3: now also JPI1.2 (Pin_2), R13.1 (Pin_1); no longer JESP1.18 (Pin_18), JPI1.5 (Pin_5)
- new net +5V_ESP_PROTECTED: D2.1 (Pin_1), F102.2 (Pin_2), JESP1.15 (Pin_15)
- new net ESP_UART_RX_3V3: JESP1.18 (Pin_18), R13.2 (Pin_2)
- new net ESP_UART_TX_3V3: JESP1.19 (Pin_19), R14.1 (Pin_1)
Changed lines of the file:
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@@
 	)
 	(symbol
-		(lib_id "RobotCarrier:Conn_01x06")
+		(lib_id "RobotCarrier:Conn_01x03")
 		(at 100.33 154.94 0)
 		(unit 1)
@@
 			)
 		)
-		(property "Value" "RPI4B POWER UART"
+		(property "Value" "RPI4B UART (GND / TX / RX)"
 			(at 100.33 158.75 0)
 				(effects
@@
 			)
 		)
-		(property "Footprint" "Custom:PI_REMOTE_1X06_MALE"
+		(property "Footprint" "Custom:DUPONT_MALE_1X03"
 			(at 100.33 154.94 0)
 				(effects
@@
 			)
 		)
-		(property "Description" "RPI4B POWER UART"
+		(property "Description" "RPI4B UART only; Raspberry Pi is powered separately"
 			(at 100.33 154.94 0)
 				(effects
@@
 		(pin "2")
 		(pin "3")
-		(pin "4")
-		(pin "5")
-		(pin "6")
 		(instances
 			(project "robot-carrier"
@@
 		)
 	)
-	(label "+5V"
+	(label "GND"
 		(at 95.25 154.94 180)
 			(effects
@@
 		)
 	)
-	(label "+5V"
+	(label "PI_UART_TX_3V3"
 		(at 95.25 157.48 180)
 			(effects
@@
 		)
 	)
-	(label "GND"
+	(label "PI_UART_RX_3V3"
 		(at 95.25 160.02 180)
-			(effects
-			(font
-				(size 1 1)
-			)
-			(justify right bottom)
-		)
-	)
-	(label "GND"
-		(at 95.25 162.56 180)
-			(effects
-			(font
-				(size 1 1)
-			)
-			(justify right bottom)
-		)
-	)
-	(label "PI_UART_TX_3V3"
-		(at 95.25 165.1 180)
-			(effects
-			(font
-				(size 1 1)
-			)
-			(justify right bottom)
-		)
-	)
-	(label "PI_UART_RX_3V3"
-		(at 95.25 167.64 180)
 			(effects
 			(font
@@
 		)
 	)
+	(label "+5V_ESP_PROTECTED"
+		(at 214.63 66.04 180)
+			(effects
+			(font
+				(size 1 1)
+			)
+			(justify right bottom)
+		)
+	)
+	(symbol
+		(lib_id "RobotCarrier:Fuse")
+		(at 160.02 66.04 0)
+		(unit 1)
+		(exclude_from_sim no)
+		(in_bom yes)
+		(on_board yes)
+		(dnp no)
+		(property "Reference" "F102"
+			(at 160.02 62.23 0)
+				(effects (font (size 1.27 1.27)))
+		)
+		(property "Value" "PPTC 0.75A 6V"
+			(at 160.02 69.85 0)
+				(effects (font (size 1.27 1.27)))
+		)
+		(property "Footprint" "Fuse:Fuse_1812_4532Metric"
+			(at 160.02 66.04 0)
+				(effects (font (size 1.27 1.27)) (hide yes))
+		)
+		(property "Datasheet" "~"
+			(at 160.02 66.04 0)
+				(effects (font (size 1.27 1.27)) (hide yes))
+		)
+		(property "Description" "Resettable fuse protecting the ESP32 5V input"
+			(at 160.02 66.04 0)
+				(effects (font (size 1.27 1.27)) (hide yes))
+		)
+		(property "LCSC" "TBD"
+			(at 160.02 66.04 0)
+				(effects (font (size 1.27 1.27)) (hide yes))
+		)
+		(pin "1")
+		(pin "2")
+		(instances
+			(project "robot-carrier"
+				(path "/00000000-0000-4000-8000-000000000001"
+					(reference "F102")
+					(unit 1)
+				)
+			)
+		)
+	)
 	(label "+5V"
-		(at 214.63 66.04 180)
-			(effects
-			(font
-				(size 1 1)
-			)
-			(justify right bottom)
-		)
+		(at 154.94 66.04 180)
+		(effects (font (size 1 1)) (justify right bottom))
+	)
+	(label "+5V_ESP_PROTECTED"
+		(at 165.1 66.04 0)
+		(effects (font (size 1 1)) (justify left bottom))
+	)
+	(symbol
+		(lib_id "RobotCarrier:D_TVS")
+		(at 160.02 76.2 0)
+		(unit 1)
+		(exclude_from_sim no)
+		(in_bom yes)
+		(on_board yes)
+		(dnp no)
+		(property "Reference" "D2"
+			(at 160.02 72.39 0)
+				(effects (font (size 1.27 1.27)))
+		)
+		(property "Value" "SMAJ5.0A"
+			(at 160.02 80.01 0)
+				(effects (font (size 1.27 1.27)))
+		)
+		(property "Footprint" "Diode_SMD:D_SMA"
+			(at 160.02 76.2 0)
+				(effects (font (size 1.27 1.27)) (hide yes))
+		)
+		(property "Datasheet" "~"
+			(at 160.02 76.2 0)
+				(effects (font (size 1.27 1.27)) (hide yes))
+		)
+		(property "Description" "5V unidirectional TVS clamp at the ESP32 input"
+			(at 160.02 76.2 0)
+				(effects (font (size 1.27 1.27)) (hide yes))
+		)
+		(property "LCSC" "TBD"
+			(at 160.02 76.2 0)
+				(effects (font (size 1.27 1.27)) (hide yes))
+		)
+		(pin "1")
+		(pin "2")
+		(instances
+			(project "robot-carrier"
+				(path "/00000000-0000-4000-8000-000000000001"
+					(reference "D2")
+					(unit 1)
+				)
+			)
+		)
+	)
+	(label "+5V_ESP_PROTECTED"
+		(at 154.94 76.2 180)
+		(effects (font (size 1 1)) (justify right bottom))
+	)
+	(label "GND"
+		(at 165.1 76.2 0)
+		(effects (font (size 1 1)) (justify left bottom))
 	)
 	(label "GND"
@@
 		)
 	)
-	(label "PI_UART_TX_3V3"
+	(label "ESP_UART_RX_3V3"
 		(at 214.63 73.66 180)
 			(effects
@@
 		)
 	)
-	(label "PI_UART_RX_3V3"
+	(label "ESP_UART_TX_3V3"
 		(at 214.63 76.2 180)
 			(effects
@@
 	(label "VIN_PROTECTED" (at 40.64 182.88 180) (effects (font (size 1 1)) (justify right bottom)))
 	(label "GND" (at 50.8 182.88 0) (effects (font (size 1 1)) (justify left bottom)))
+	(symbol
+		(lib_id "RobotCarrier:R")
+		(at 299.72 116.84 0)
+		(unit 1)
+		(exclude_from_sim no)
+		(in_bom yes)
+		(on_board yes)
+		(dnp no)
+		(property "Reference" "R13" (at 299.72 113.03 0) (effects (font (size 1.27 1.27))))
+		(property "Value" "470R" (at 299.72 120.65 0) (effects (font (size 1.27 1.27))))
+		(property "Footprint" "Custom:R_1206_HAND" (at 299.72 116.84 0) (effects (font (size 1.27 1.27)) (hide yes)))
+		(property "Datasheet" "~" (at 299.72 116.84 0) (effects (font (size 1.27 1.27)) (hide yes)))
+		(property "Description" "Pi TX to ESP32 RX UART series resistor" (at 299.72 116.84 0) (effects (font (size 1.27 1.27)) (hide yes)))
+		(property "LCSC" "TBD" (at 299.72 116.84 0) (effects (font (size 1.27 1.27)) (hide yes)))
+		(pin "1")
+		(pin "2")
+		(instances (project "robot-carrier" (path "/00000000-0000-4000-8000-000000000001" (reference "R13") (unit 1))))
+	)
+	(label "PI_UART_TX_3V3" (at 294.64 116.84 180) (effects (font (size 1 1)) (justify right bottom)))
+	(label "ESP_UART_RX_3V3" (at 304.8 116.84 0) (effects (font (size 1 1)) (justify left bottom)))
+	(symbol
+		(lib_id "RobotCarrier:R")
+		(at 299.72 127 0)
+		(unit 1)
+		(exclude_from_sim no)
+		(in_bom yes)
+		(on_board yes)
+		(dnp no)
+		(property "Reference" "R14" (at 299.72 123.19 0) (effects (font (size 1.27 1.27))))
+		(property "Value" "470R" (at 299.72 130.81 0) (effects (font (size 1.27 1.27))))
+		(property "Footprint" "Custom:R_1206_HAND" (at 299.72 127 0) (effects (font (size 1.27 1.27)) (hide yes)))
+		(property "Datasheet" "~" (at 299.72 127 0) (effects (font (size 1.27 1.27)) (hide yes)))
+		(property "Description" "ESP32 TX to Pi RX UART series resistor" (at 299.72 127 0) (effects (font (size 1.27 1.27)) (hide yes)))
+		(property "LCSC" "TBD" (at 299.72 127 0) (effects (font (size 1.27 1.27)) (hide yes)))
+		(pin "1")
+		(pin "2")
+		(instances (project "robot-carrier" (path "/00000000-0000-4000-8000-000000000001" (reference "R14") (unit 1))))
+	)
+	(label "ESP_UART_TX_3V3" (at 294.64 127 180) (effects (font (size 1 1)) (justify right bottom)))
+	(label "PI_UART_RX_3V3" (at 304.8 127 0) (effects (font (size 1 1)) (justify left bottom)))
 	(sheet_instances
 		(path "/"
